File: KiCad/r1.kicad_pcb (KiCad board)
At the start: 2 copper layers, 215.9 x 127 mm, 68 parts, among them J1 KEYBOARD, J3 ATX-20, J4 DE9_Socket, J5 R1 EXPANSION, Q1 2N4401, SW1 RESET, U1 6502, U10 74LS245, U11 MAX232, U2 6821, U3 27C64, U4 HM62256BLP, U5 74LS138, U6 74LS00, U7 74LS04, U8 P8X32A-D40, U9 24LC256, X1 1 MHz, X2 5MHz

Commit message: Unzipped and rearranged directories
Parts:
- added C21: 100, Capacitor_THT:CP_Radial_D10.0mm_P5.00mm, F.Cu at (54.6, -180.3)
- added C22: 100, Capacitor_THT:CP_Radial_D5.0mm_P2.50mm, F.Cu at (46.0, -185.4)
- added D1: POWER, LED_THT:LED_D5.0mm, F.Cu at (88.9, -182.9)
- added JP1: SolderJumper_2_Open, TestPoint:TestPoint_Bridge_Pitch2.54mm_Drill1.0mm, F.Cu at (141.0, -116.8)
- added JP2: SolderJumper_2_Open, TestPoint:TestPoint_Bridge_Pitch2.54mm_Drill1.0mm, F.Cu at (217.2, -161.3)
- added S1: ON/OFF, Button_Switch_THT:SW_PUSH_6mm, F.Cu at (283.0, -142.7)
- added S3: CLEAR, Button_Switch_THT:SW_PUSH_6mm, F.Cu at (283.0, -134.2)
- renumbered SW1 to S2
Connections:
- C13 pad 1: unconnected-(C13-Pad1) -> Net-(C13-Pad1)
- C13 pad 2: unconnected-(C13-Pad2) -> Net-(C13-Pad2)
- C14 pad 1: unconnected-(C14-Pad1) -> /VCC
- C14 pad 2: unconnected-(C14-Pad2) -> GND
- C15 pad 1: unconnected-(C15-Pad1) -> /VDD
- C15 pad 2: unconnected-(C15-Pad2) -> GND
- C16 pad 1: unconnected-(C16-Pad1) -> Net-(U11-C1+)
- C16 pad 2: unconnected-(C16-Pad2) -> Net-(U11-C1-)
- C17 pad 1: unconnected-(C17-Pad1) -> Net-(U11-C2+)
- C17 pad 2: unconnected-(C17-Pad2) -> Net-(U11-C2-)
- C18 pad 1: unconnected-(C18-Pad1) -> Net-(U11-VS+)
- C18 pad 2: unconnected-(C18-Pad2) -> /VCC
- C19 pad 1: unconnected-(C19-Pad1) -> GND
- C19 pad 2: unconnected-(C19-Pad2) -> Net-(U11-VS-)
- C20 pad 1: unconnected-(C20-Pad1) -> /VCC
- C20 pad 2: unconnected-(C20-Pad2) -> GND
- C8 pad 1: /VDD -> GND
- C8 pad 2: GND -> /VDD
- C9 pad 1: /VDD -> GND
- C9 pad 2: GND -> /VDD
- J3 pad 1: Net-(J3-+3.3V-Pad1) -> unconnected-(J3-+3.3V-Pad1)
- J3 pad 10: unconnected-(J3-+12V-Pad10) -> /12V
- J3 pad 11: Net-(J3-+3.3V-Pad1) -> unconnected-(J3-+3.3V-Pad1)_2
- J3 pad 12: unconnected-(J3--12V-Pad12) -> /-12V
- J3 pad 13: Net-(J3-GND-Pad13) -> GND
- J3 pad 14: unconnected-(J3-PS_ON#-Pad14) -> Net-(J3-PS_ON#)
- J3 pad 15: Net-(J3-GND-Pad13) -> GND
- J3 pad 16: Net-(J3-GND-Pad13) -> GND
- J3 pad 17: Net-(J3-GND-Pad13) -> GND
- J3 pad 19: Net-(J3-+5V-Pad19) -> /VCC
- J3 pad 2: Net-(J3-+3.3V-Pad1) -> unconnected-(J3-+3.3V-Pad1)_1
- J3 pad 20: Net-(J3-+5V-Pad19) -> /VCC
- J3 pad 3: Net-(J3-GND-Pad13) -> GND
- J3 pad 4: Net-(J3-+5V-Pad19) -> /VCC
- J3 pad 5: Net-(J3-GND-Pad13) -> GND
- J3 pad 6: Net-(J3-+5V-Pad19) -> /VCC
- J3 pad 7: Net-(J3-GND-Pad13) -> GND
- J4 pad 1: unconnected-(J4-Pad1) -> Net-(J4-Pad1)
- J4 pad 2: unconnected-(J4-Pad2) -> Net-(U11-T1OUT)
- J4 pad 3: unconnected-(J4-Pad3) -> Net-(U11-R1IN)
- J4 pad 4: unconnected-(J4-Pad4) -> Net-(C13-Pad1)
- J4 pad 5: unconnected-(J4-Pad5) -> GND
- J4 pad 6: unconnected-(J4-Pad6) -> Net-(J4-Pad1)
- J5 pad 1: unconnected-(J5-Pin_1-Pad1) -> /-12V
- J5 pad 10: unconnected-(J5-Pin_10-Pad10) -> /A12
- J5 pad 11: unconnected-(J5-Pin_11-Pad11) -> /A14
- J5 pad 12: unconnected-(J5-Pin_12-Pad12) -> /R/W
- J5 pad 13: unconnected-(J5-Pin_13-Pad13) -> /$A000
- J5 pad 14: unconnected-(J5-Pin_14-Pad14) -> /PHI1
- J5 pad 15: unconnected-(J5-Pin_15-Pad15) -> /D1
- J5 pad 16: unconnected-(J5-Pin_16-Pad16) -> /D3
- J5 pad 17: unconnected-(J5-Pin_17-Pad17) -> /D5
- J5 pad 18: unconnected-(J5-Pin_18-Pad18) -> /D7
- J5 pad 19: unconnected-(J5-Pin_19-Pad19) -> /SYNC
- J5 pad 2: unconnected-(J5-Pin_2-Pad2) -> /12V
- J5 pad 20: unconnected-(J5-Pin_20-Pad20) -> /PHI2
- J5 pad 21: unconnected-(J5-Pin_21-Pad21) -> /VCC
- J5 pad 22: unconnected-(J5-Pin_22-Pad22) -> /$C000
- J5 pad 23: unconnected-(J5-Pin_23-Pad23) -> /PHI0
- J5 pad 24: unconnected-(J5-Pin_24-Pad24) -> /A1
- J5 pad 25: unconnected-(J5-Pin_25-Pad25) -> /A3
- J5 pad 26: unconnected-(J5-Pin_26-Pad26) -> /A5
- J5 pad 27: unconnected-(J5-Pin_27-Pad27) -> /A7
- J5 pad 28: unconnected-(J5-Pin_28-Pad28) -> /A9
- J5 pad 29: unconnected-(J5-Pin_29-Pad29) -> /A11
- J5 pad 3: unconnected-(J5-Pin_3-Pad3) -> GND
- J5 pad 30: unconnected-(J5-Pin_30-Pad30) -> /A13
- J5 pad 31: unconnected-(J5-Pin_31-Pad31) -> /A15
- J5 pad 32: unconnected-(J5-Pin_32-Pad32) -> /$B000
- J5 pad 33: unconnected-(J5-Pin_33-Pad33) -> /D0
- J5 pad 34: unconnected-(J5-Pin_34-Pad34) -> /D2
- J5 pad 35: unconnected-(J5-Pin_35-Pad35) -> /D4
- J5 pad 36: unconnected-(J5-Pin_36-Pad36) -> /D6
- J5 pad 37: unconnected-(J5-Pin_37-Pad37) -> /RDY
- J5 pad 38: unconnected-(J5-Pin_38-Pad38) -> /IRQ
- J5 pad 39: unconnected-(J5-Pin_39-Pad39) -> /NMI
- J5 pad 4: unconnected-(J5-Pin_4-Pad4) -> /A0
- J5 pad 40: unconnected-(J5-Pin_40-Pad40) -> /RESET
- J5 pad 5: unconnected-(J5-Pin_5-Pad5) -> /A2
- J5 pad 6: unconnected-(J5-Pin_6-Pad6) -> /A4
- J5 pad 7: unconnected-(J5-Pin_7-Pad7) -> /A6
- J5 pad 8: unconnected-(J5-Pin_8-Pad8) -> /A8
- J5 pad 9: unconnected-(J5-Pin_9-Pad9) -> /A10
- Q1 pad 1: unconnected-(Q1-C-Pad1) -> /RST
- Q1 pad 2: unconnected-(Q1-B-Pad2) -> Net-(Q1-B)
- Q1 pad 3: unconnected-(Q1-E-Pad3) -> GND
- R18 pad 1: Net-(J2-In) -> /RX
- R18 pad 2: Net-(U8-P13) -> Net-(U11-R1OUT)
- R19 pad 1: Net-(J2-In) -> unconnected-(R19-Pad1)
- R19 pad 2: Net-(U8-P14) -> unconnected-(R19-Pad2)
- R20 pad 1: unconnected-(R20-Pad1) -> Net-(D1-K)
- R20 pad 2: unconnected-(R20-Pad2) -> /VCC
- R21 pad 1: unconnected-(R21-Pad1) -> Net-(J2-In)
- R21 pad 2: unconnected-(R21-Pad2) -> Net-(U8-P14)
- R23 pad 1: unconnected-(R23-Pad1) -> Net-(U8-P13)
- R23 pad 2: unconnected-(R23-Pad2) -> Net-(J2-In)
- R24 pad 1: unconnected-(R24-Pad1) -> Net-(Q1-B)
- R24 pad 2: unconnected-(R24-Pad2) -> GND
- R25 pad 1: unconnected-(R25-Pad1) -> Net-(C13-Pad2)
- R25 pad 2: unconnected-(R25-Pad2) -> Net-(Q1-B)
- R6 pad 1: Net-(U8-P29) -> /VDD
- R6 pad 2: /VDD -> Net-(U8-P29)
- U11 pad 1: unconnected-(U11-C1+-Pad1) -> Net-(U11-C1+)
- U11 pad 11: unconnected-(U11-T1IN-Pad11) -> /TX
- U11 pad 12: unconnected-(U11-R1OUT-Pad12) -> Net-(U11-R1OUT)
- U11 pad 13: unconnected-(U11-R1IN-Pad13) -> Net-(U11-R1IN)
- U11 pad 14: unconnected-(U11-T1OUT-Pad14) -> Net-(U11-T1OUT)
- U11 pad 15: unconnected-(U11-GND-Pad15) -> GND
- U11 pad 16: unconnected-(U11-VCC-Pad16) -> /VCC
- U11 pad 2: unconnected-(U11-VS+-Pad2) -> Net-(U11-VS+)
- U11 pad 3: unconnected-(U11-C1--Pad3) -> Net-(U11-C1-)
- U11 pad 4: unconnected-(U11-C2+-Pad4) -> Net-(U11-C2+)
- U11 pad 5: unconnected-(U11-C2--Pad5) -> Net-(U11-C2-)
- U11 pad 6: unconnected-(U11-VS--Pad6) -> Net-(U11-VS-)
- U3 pad 10: unconnected-(U3-A0-Pad10) -> /A0
- U3 pad 11: unconnected-(U3-D0-Pad11) -> /D0
- U3 pad 12: unconnected-(U3-D1-Pad12) -> /D1
- U3 pad 13: unconnected-(U3-D2-Pad13) -> /D2
- U3 pad 15: unconnected-(U3-D3-Pad15) -> /D3
- U3 pad 16: unconnected-(U3-D4-Pad16) -> /D4
- U3 pad 17: unconnected-(U3-D5-Pad17) -> /D5
- U3 pad 18: unconnected-(U3-D6-Pad18) -> /D6
- U3 pad 19: unconnected-(U3-D7-Pad19) -> /D7
- U3 pad 2: unconnected-(U3-A12-Pad2) -> /A12
- U3 pad 20: unconnected-(U3-~{CE}-Pad20) -> Net-(U3-~{CE})
- U3 pad 21: unconnected-(U3-A10-Pad21) -> /A10
- U3 pad 22: unconnected-(U3-~{OE}-Pad22) -> Net-(U3-~{CE})
- U3 pad 23: unconnected-(U3-A11-Pad23) -> /A11
- U3 pad 24: unconnected-(U3-A9-Pad24) -> /A9
- U3 pad 25: unconnected-(U3-A8-Pad25) -> /A8
- U3 pad 27: unconnected-(U3-~{PGM}-Pad27) -> /VCC
- U3 pad 28: unconnected-(U3-VCC-Pad28) -> /VCC
- U3 pad 3: unconnected-(U3-A7-Pad3) -> /A7
- U3 pad 4: unconnected-(U3-A6-Pad4) -> /A6
- U3 pad 5: unconnected-(U3-A5-Pad5) -> /A5
- U3 pad 6: unconnected-(U3-A4-Pad6) -> /A4
- U3 pad 7: unconnected-(U3-A3-Pad7) -> /A3
- U3 pad 8: unconnected-(U3-A2-Pad8) -> /A2
- U3 pad 9: unconnected-(U3-A1-Pad9) -> /A1
- U4 pad 1: unconnected-(U4-A14-Pad1) -> /A14
- U4 pad 10: unconnected-(U4-A0-Pad10) -> /A0
- U4 pad 11: unconnected-(U4-Q0-Pad11) -> /D0
- U4 pad 12: unconnected-(U4-Q1-Pad12) -> /D1
- U4 pad 13: unconnected-(U4-Q2-Pad13) -> /D2
- U4 pad 15: unconnected-(U4-Q3-Pad15) -> /D3
- U4 pad 16: unconnected-(U4-Q4-Pad16) -> /D4
- U4 pad 17: unconnected-(U4-Q5-Pad17) -> /D5
- U4 pad 18: unconnected-(U4-Q6-Pad18) -> /D6
- U4 pad 19: unconnected-(U4-Q7-Pad19) -> /D7
- U4 pad 2: unconnected-(U4-A12-Pad2) -> /A12
- U4 pad 20: unconnected-(U4-~{CS}-Pad20) -> /A15
- U4 pad 21: unconnected-(U4-A10-Pad21) -> /A10
- U4 pad 22: unconnected-(U4-~{OE}-Pad22) -> /A15
- U4 pad 23: unconnected-(U4-A11-Pad23) -> /A11
- U4 pad 24: unconnected-(U4-A9-Pad24) -> /A9
- U4 pad 25: unconnected-(U4-A8-Pad25) -> /A8
- U4 pad 26: unconnected-(U4-A13-Pad26) -> /A13
- U4 pad 27: unconnected-(U4-~{WE}-Pad27) -> Net-(U4-~{WE})
- U4 pad 28: unconnected-(U4-VCC-Pad28) -> /VCC
- U4 pad 3: unconnected-(U4-A7-Pad3) -> /A7
- U4 pad 4: unconnected-(U4-A6-Pad4) -> /A6
- U4 pad 5: unconnected-(U4-A5-Pad5) -> /A5
- U4 pad 6: unconnected-(U4-A4-Pad6) -> /A4
- U4 pad 7: unconnected-(U4-A3-Pad7) -> /A3
- U4 pad 8: unconnected-(U4-A2-Pad8) -> /A2
- U4 pad 9: unconnected-(U4-A1-Pad9) -> /A1
- U5 pad 1: unconnected-(U5-A0-Pad1) -> /A12
- U5 pad 10: unconnected-(U5-O5-Pad10) -> /$D000
- U5 pad 11: unconnected-(U5-O4-Pad11) -> /$C000
- U5 pad 12: unconnected-(U5-O3-Pad12) -> /$B000
- U5 pad 13: unconnected-(U5-O2-Pad13) -> /$A000
- U5 pad 16: unconnected-(U5-VCC-Pad16) -> /VCC
- U5 pad 2: unconnected-(U5-A1-Pad2) -> /A13
- U5 pad 3: unconnected-(U5-A2-Pad3) -> /A14
- U5 pad 4: unconnected-(U5-E1-Pad4) -> GND
- U5 pad 5: unconnected-(U5-E2-Pad5) -> GND
- U5 pad 6: unconnected-(U5-E3-Pad6) -> /A15
- U5 pad 7: unconnected-(U5-O7-Pad7) -> Net-(U5-O7)
- U5 pad 8: unconnected-(U5-GND-Pad8) -> GND
- U5 pad 9: unconnected-(U5-O6-Pad9) -> Net-(U5-O6)
- U6 pad 1: unconnected-(U6-Pad1) -> Net-(U5-O6)
- U6 pad 10: unconnected-(U6-Pad10) -> Net-(U6-Pad10)
- U6 pad 11: unconnected-(U6-Pad11) -> Net-(U4-~{WE})
- U6 pad 12: unconnected-(U6-Pad12) -> /PHI2
- U6 pad 13: unconnected-(U6-Pad13) -> Net-(U6-Pad13)
- U6 pad 2: unconnected-(U6-Pad2) -> Net-(U5-O7)
- U6 pad 3: unconnected-(U6-Pad3) -> Net-(U6-Pad10)
- U6 pad 4: unconnected-(U6-Pad4) -> /R/W
- U6 pad 5: unconnected-(U6-Pad5) -> /R/W
- U6 pad 6: unconnected-(U6-Pad6) -> Net-(U6-Pad13)
- U6 pad 8: unconnected-(U6-Pad8) -> Net-(U3-~{CE})
- U6 pad 9: unconnected-(U6-Pad9) -> Net-(U6-Pad10)
- U8 pad 11: Net-(JP2-B) -> /RST
- V1 pad 1: unconnected-(V1-VI-Pad1) -> Net-(V1-VI)
- V1 pad 2: unconnected-(V1-GND-Pad2) -> GND
- V1 pad 3: unconnected-(V1-VO-Pad3) -> /VCC
- V2 pad 1: unconnected-(V2-IN-Pad1) -> /VCC
- V2 pad 2: unconnected-(V2-GND-Pad2) -> GND
- V2 pad 3: unconnected-(V2-OUT-Pad3) -> /VDD
Routing:
- net (no net): track 2803.8 -> 10338.8 mm, vias 184 -> 176
- net /VCC: track 0.00 -> 562.3 mm, vias 0 -> 3
- net unconnected-(U5-VCC-Pad16): track 528.9 -> 0.00 mm, vias 2 -> 0
- net unconnected-(U5-A0-Pad1): track 406.9 -> 0.00 mm, vias 3 -> 0
- net unconnected-(U5-A1-Pad2): track 404.4 -> 0.00 mm, vias 5 -> 0
- net GND: track 122.1 -> 518.5 mm, vias 1 -> 5
- net unconnected-(U3-A3-Pad7): track 379.5 -> 0.00 mm, vias 7 -> 0
- net unconnected-(U3-D0-Pad11): track 375.7 -> 0.00 mm, vias 1 -> 0
- net unconnected-(U3-A5-Pad5): track 373.5 -> 0.00 mm, vias 5 -> 0
- net unconnected-(U5-A2-Pad3): track 349.2 -> 0.00 mm, vias 4 -> 0
- net unconnected-(U3-A7-Pad3): track 348.2 -> 0.00 mm, vias 4 -> 0
- net unconnected-(U3-D6-Pad18): track 345.0 -> 0.00 mm, vias 4 -> 0
- net unconnected-(U3-D3-Pad15): track 336.3 -> 0.00 mm, vias 4 -> 0
- net unconnected-(U3-A10-Pad21): track 332.5 -> 0.00 mm, vias 4 -> 0
- net unconnected-(U3-A1-Pad9): track 331.0 -> 0.00 mm, vias 5 -> 0
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
Commit message: R20260909
Connections:
- R19 pad 1: unconnected-(R19-Pad1) -> /KCL
- R19 pad 2: unconnected-(R19-Pad2) -> Net-(J6-Pad5)
- R20 pad 1: Net-(D1-K) -> Net-(J6-Pad1)
- R20 pad 2: /VCC -> /DATA
- R22 pad 1: unconnected-(R22-Pad1) -> /VCC
- R22 pad 2: unconnected-(R22-Pad2) -> Net-(D1-K)
- R25 pad 1: Net-(C13-Pad2) -> Net-(Q1-B)
- R25 pad 2: Net-(Q1-B) -> Net-(C13-Pad2)
- R7 pad 1: unconnected-(R7-Pad1) -> /VDD
- R7 pad 2: unconnected-(R7-Pad2) -> Net-(J6-Pad5)
- R8 pad 1: unconnected-(R8-Pad1) -> /VDD
- R8 pad 2: unconnected-(R8-Pad2) -> Net-(J6-Pad1)
Routing:
- net (no net): track 10338.8 -> 9718.6 mm
- net /A2: track 0.00 -> 238.4 mm
- net GND: track 518.5 -> 653.0 mm
- net /VCC: track 562.3 -> 682.5 mm
- net /VDD: track 240.8 -> 346.7 mm
- net unconnected-(R22-Pad2): track 60.0 -> 0.00 mm, vias 1 -> 0
- net Net-(D1-K): track 0.00 -> 60.0 mm, vias 0 -> 1
- net Net-(Q1-B): track 0.00 -> 16.1 mm
- net unconnected-(R7-Pad2): track 15.0 -> 0.00 mm, vias 1 -> 0
- net Net-(J6-Pad5): track 0.00 -> 15.0 mm, vias 0 -> 1
- net Net-(C13-Pad2): track 0.00 -> 4.86 mm
- net Net-(J4-Pad1): track 3.41 -> 4.46 mm

Commit message: R20260910
Parts:
- added J7: 7-9V DC, Connector_BarrelJack:BarrelJack_GCT_DCJ200-10-A_Horizontal, F.Cu at (77.5, -189.3)
- added REF**: breadboard, r1te:breadboard, F.Cu at (120.7, -172.7)
- added REF**: Symbol_Barrel_Polarity, Symbol:Symbol_Barrel_Polarity, F.Cu at (77.5, -185.0)
- C22: footprint Capacitor_THT:CP_Radial_D5.0mm_P2.50mm -> Capacitor_THT:CP_Radial_D5.0mm_P2.00mm
- moved S1 231.1 mm to (62.1, -210.9)
- moved C22 204.0 mm to (249.9, -191.0)
- moved S3 83.2 mm to (205.7, -165.1)
Connections:
- net /-12V renamed -12V
- net /VDD renamed VDD
- C1 pad 2: /VCC -> VCC
- C10 pad 2: /VCC -> VCC
- C11 pad 2: /VCC -> VCC
- C12 pad 2: /VCC -> VCC
- C14 pad 1: /VCC -> VCC
- C18 pad 2: /VCC -> VCC
- C2 pad 2: /VCC -> VCC
- C20 pad 1: /VCC -> VCC
- C3 pad 2: /VCC -> VCC
- C4 pad 2: /VCC -> VCC
- C5 pad 2: /VCC -> VCC
- C6 pad 2: /VCC -> VCC
- C7 pad 2: /VCC -> VCC
- J1 pad 1: /VCC -> VCC
- J3 pad 10: /12V -> +12V
- J3 pad 19: /VCC -> VCC
- J3 pad 20: /VCC -> VCC
- J3 pad 4: /VCC -> VCC
- J3 pad 6: /VCC -> VCC
- J5 pad 10: /A12 -> /A3
- J5 pad 11: /A14 -> /A4
- J5 pad 12: /R/W -> /A5
- J5 pad 13: /$A000 -> /A6
- J5 pad 14: /PHI1 -> /A7
- J5 pad 15: /D1 -> /A8
- J5 pad 16: /D3 -> /A9
- J5 pad 17: /D5 -> /A10
- J5 pad 18: /D7 -> /A11
- J5 pad 19: /SYNC -> /A12
- J5 pad 2: /12V -> VCC
- J5 pad 20: /PHI2 -> /A13
- J5 pad 21: /VCC -> /A14
- J5 pad 22: /$C000 -> /A15
- J5 pad 23: /PHI0 -> /R/W
- J5 pad 24: /A1 -> /$B000
- J5 pad 25: /A3 -> /$A000
- J5 pad 26: /A5 -> /D0
- J5 pad 27: /A7 -> /PHI1
- J5 pad 28: /A9 -> /D2
- J5 pad 29: /A11 -> /D1
- J5 pad 3: GND -> +12V
- J5 pad 30: /A13 -> /D4
- J5 pad 31: /A15 -> /D3
- J5 pad 32: /$B000 -> /D6
- J5 pad 33: /D0 -> /D5
- J5 pad 34: /D2 -> /RDY
- J5 pad 35: /D4 -> /D7
- J5 pad 36: /D6 -> /IRQ
- J5 pad 37: /RDY -> /SYNC
- J5 pad 38: /IRQ -> /NMI
- J5 pad 39: /NMI -> /PHI2
- J5 pad 4: /A0 -> /$C000
- J5 pad 5: /A2 -> GND
- J5 pad 6: /A4 -> /PHI0
- J5 pad 7: /A6 -> /A0
- J5 pad 8: /A8 -> /A1
- J5 pad 9: /A10 -> /A2
- R1 pad 1: /VCC -> VCC
- R18 pad 1: /RX -> Net-(U11-R1OUT)
- R18 pad 2: Net-(U11-R1OUT) -> /RX
- R2 pad 1: /VCC -> VCC
- R20 pad 1: Net-(J6-Pad1) -> /DATA
- R20 pad 2: /DATA -> Net-(J6-Pad1)
- R22 pad 1: /VCC -> VCC
- R23 pad 1: Net-(U8-P13) -> Net-(J2-In)
- R23 pad 2: Net-(J2-In) -> Net-(U8-P13)
- R26 pad 1: /STROBE -> GND
- R26 pad 2: GND -> /STROBE
- R3 pad 1: /VCC -> VCC
- R4 pad 1: /VCC -> VCC
- R5 pad 1: unconnected-(R5-Pad1) -> /K7
- R5 pad 2: unconnected-(R5-Pad2) -> GND
- S2 pad 1: /RESET -> GND
- S2 pad 2: GND -> /RESET
- U1 pad 8: /VCC -> VCC
- U10 pad 1: /VCC -> VCC
- U10 pad 20: /VCC -> VCC
- U11 pad 16: /VCC -> VCC
- U2 pad 20: /VCC -> VCC
- U2 pad 24: /VCC -> VCC
- U3 pad 27: /VCC -> VCC
- U3 pad 28: /VCC -> VCC
- U4 pad 28: /VCC -> VCC
- U5 pad 16: /VCC -> VCC
- U6 pad 14: unconnected-(U6E-VCC-Pad14) -> VCC
- U6 pad 7: unconnected-(U6E-GND-Pad7) -> GND
- U7 pad 14: unconnected-(U7G-VCC-Pad14) -> VCC
- U7 pad 7: unconnected-(U7G-GND-Pad7) -> GND
- V1 pad 3: /VCC -> VCC
- V2 pad 1: /VCC -> VCC
- X1 pad 14: unconnected-(X1-Vcc-Pad14) -> VCC
- X1 pad 7: unconnected-(X1-GND-Pad7) -> GND
Routing:
- net (no net): track 9718.6 -> 1105.9 mm, vias 176 -> 15
- net /VCC: track 682.5 -> 0.00 mm, vias 3 -> 0
- net VCC: track 0.00 -> 671.1 mm, vias 0 -> 10
- net unconnected-(U6E-VCC-Pad14): track 469.5 -> 0.00 mm, vias 8 -> 0
- net /A12: track 0.00 -> 402.4 mm
- net /A4: track 0.00 -> 389.4 mm, vias 0 -> 3
- net /A3: track 0.00 -> 373.8 mm, vias 11 -> 7
- net /A5: track 0.00 -> 367.1 mm
- net /D0: track 0.00 -> 365.6 mm
- net /A7: track 0.00 -> 346.8 mm
- net /A14: track 0.00 -> 344.2 mm
- net /A10: track 0.00 -> 329.9 mm
- net /D3: track 7.10 -> 333.8 mm
- net /A1: track 0.00 -> 324.4 mm, vias 8 -> 5
- net /D5: track 0.00 -> 322.7 mm
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
Commit message: R20260918
Parts:
- removed R27: 1K, Resistor_THT:R_Axial_DIN0207_L6.3mm_D2.5mm_P10.16mm_Horizontal
- removed the REF** at (77.5, -185.0)
- added J2: VIDEO OUT, r1te:Keystone 901, F.Cu at (132.1, -195.7)
- JP1, JP2: value SolderJumper_2_Open -> Jumper_2_Open
- S1: footprint Button_Switch_THT:SW_PUSH_6mm -> r1te:ToggleSW_DPDT_VerticalPC
- U6: footprint Package_DIP:DIP-16_W7.62mm_Socket_LongPads -> Package_DIP:DIP-14_W7.62mm_Socket_LongPads
- moved S1 17.5 mm to (64.6, -228.2)
Connections:
- J7 pad 1: unconnected-(J7-Pad1) -> Net-(J7-Pad1)
- J7 pad 2: unconnected-(J7-Pad2) -> GND
- J7 pad 3: (no net) -> GND
- R10 pad 1: Net-(U8-P1) -> /PB1
- R10 pad 2: /PB1 -> Net-(U8-P1)
- U2 pad 10: unconnected-(U2-PB0-Pad10) -> /PB0
- U2 pad 23: /$D00 -> /$D000
- X1 pad 8: unconnected-(X1-OUT-Pad8) -> /PHI0
- X2 pad 1: Net-(U8-XI) -> Net-(U8-XO)
- X2 pad 2: Net-(U8-XO) -> Net-(U8-XI)
Routing:
- net (no net): track 1105.9 -> 13.5 mm, vias 15 -> 9
- net /PHI2: track 0.00 -> 468.4 mm, vias 0 -> 8
- net GND: track 895.0 -> 1130.2 mm
- net /RST: track 13.4 -> 167.5 mm
- net /$D000: track 0.00 -> 77.5 mm, vias 0 -> 4
- net /$D00: track 77.5 -> 0.00 mm, vias 4 -> 0
- net unconnected-(U2-PB0-Pad10): track 72.1 -> 0.00 mm, vias 3 -> 0
- net /PB0: track 0.00 -> 72.1 mm, vias 0 -> 3
- net Net-(U3-~{CE}): track 0.00 -> 68.0 mm, vias 0 -> 1
- net VCC: track 671.1 -> 726.1 mm, vias 10 -> 2
- net Net-(U4-~{WE}): track 0.00 -> 42.2 mm
- net unconnected-(U11-R2OUT-Pad9): track 40.0 -> 0.00 mm, vias 1 -> 0
- net Net-(U8-XI): track 0.00 -> 26.1 mm, vias 0 -> 1
- net Net-(U8-XO): track 0.00 -> 21.7 mm, vias 0 -> 1
- net unconnected-(J7-Pad1): track 13.7 -> 0.00 mm, vias 1 -> 0
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